File: Sensors/Temperatuur/PT1000_sensor/PT1000_sensor.kicad_pcb (KiCad board)
At the start: 2 copper layers, 18 parts, among them Q1 BC546, U1 LTC2055

Commit message: created a pcb and sends it of
Parts:
- added C10: 100nF, Capacitor_SMD:C_0805_2012Metric, F.Cu at (199.3, 81.9)
- added C9: 100nF, Capacitor_SMD:C_0805_2012Metric, F.Cu at (205.3, 71.3)
- added J1: Conn_01x02_Pin, Connector_PinSocket_2.54mm:PinSocket_1x02_P2.54mm_Vertical, F.Cu at (193.0, 70.5)
- added J2: Conn_01x02_Pin, Connector_PinSocket_2.54mm:PinSocket_1x02_P2.54mm_Vertical, F.Cu at (193.0, 76.0)
- added J3: Conn_01x02_Pin, Connector_PinSocket_2.54mm:PinSocket_1x02_P2.54mm_Vertical, F.Cu at (194.0, 86.0)
- added R4: 160K, Resistor_SMD:R_0805_2012Metric, F.Cu at (195.3, 82.3)
- added R6: 62, Resistor_SMD:R_0805_2012Metric, F.Cu at (217.3, 79.3)
- added R7: 510, Resistor_SMD:R_0805_2012Metric, F.Cu at (214.6, 66.3)
- added REF**: MountingHole_2.2mm_M2, MountingHole:MountingHole_2.2mm_M2, F.Cu at (199.0, 63.0)
- C3, C4: footprint Capacitor_THT:CP_Radial_D4.0mm_P2.00mm -> Capacitor_THT:CP_Radial_D4.0mm_P1.50mm
- R1: value 972 -> 910
- R3: value 16.5k -> 16k
- TH1: footprint Connector_PinHeader_1.00mm:PinHeader_1x02_P1.00mm_Vertical -> Connector_PinSocket_2.54mm:PinSocket_1x02_P2.54mm_Vertical
- moved C8 165.1 mm to (217.3, 67.3)
- moved C5 154.7 mm to (207.3, 63.3), turned to 180 degrees
- moved C7 151.3 mm to (204.3, 76.5)
- moved R3 150.7 mm to (212.6, 66.3), turned to -90 degrees
- moved ISL1 147.6 mm to (204.2, 85.4), turned to 180 degrees
- moved C6 147.4 mm to (200.3, 85.3), turned to 90 degrees
- moved R2 147.2 mm to (210.3, 76.5), turned to 180 degrees
- moved C1 143.2 mm to (204.3, 82.3), turned to 180 degrees
- moved C3 141.2 mm to (197.7, 70.4)
- moved C4 140.1 mm to (197.3, 76.0), turned to -90 degrees
- moved TH1 136.8 mm to (216.0, 82.5)
- moved U1 136.4 mm to (204.3, 79.5)
- moved Q1 136.3 mm to (211.3, 81.8)
- moved R1 133.3 mm to (217.3, 76.5), turned to 180 degrees
- moved AD1 127.5 mm to (217.3, 71.5), turned to 90 degrees
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Connections:
- AD2 pad 7: unconnected-(AD2-Pad7) -> Net-(AD2-Pad7)
- C6 pad 1: +3.3V -> +5V
- R1 pad 1: Net-(AD1-Rg-Pad2) -> Net-(R1-Pad1)
- R1 pad 2: Net-(AD1-Rg-Pad3) -> Net-(AD1-Rg-Pad2)
- R3 pad 1: Net-(AD2-Rg-Pad2) -> Net-(R3-Pad1)
- R3 pad 2: Net-(AD2-Rg-Pad3) -> Net-(AD2-Rg-Pad2)
- U1 pad 5: unconnected-(U1B-+-Pad5) -> Net-(U1B-+)
- U1 pad 6: unconnected-(U1B---Pad6) -> Net-(J3-Pin_2)
- U1 pad 7: unconnected-(U1-Pad7) -> Net-(J3-Pin_2)
Routing:
- net +5V: track 0.00 -> 88.5 mm
- net +3.3V: track 0.00 -> 38.7 mm
- net GND: track 0.00 -> 38.7 mm, vias 0 -> 5
- net Net-(AD2-Pad7): track 0.00 -> 23.4 mm, vias 0 -> 2
- net /-V_s: track 0.00 -> 20.4 mm
- net Net-(AD2-+): track 0.00 -> 12.2 mm
- net Net-(AD1-Rg-Pad3): track 0.00 -> 11.6 mm
- net +2.048V: track 0.00 -> 10.7 mm
- net Net-(J3-Pin_2): track 0.00 -> 10.1 mm
- net Net-(U1B-+): track 0.00 -> 7.97 mm
- net Net-(Q1-E): track 0.00 -> 7.90 mm
- net +1.024V: track 0.00 -> 6.23 mm
- net Net-(Q1-B): track 0.00 -> 4.90 mm
- net Net-(AD2-Rg-Pad3): track 0.00 -> 4.82 mm
- net Net-(AD1-Rg-Pad2): track 0.00 -> 3.13 mm
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- added copper zone on B.Cu, net GND
Other:
- board outline added: 31 x 30 mm
- board text added: "N.L."
