File: Sensors/Temperatuur/PT1000_sensor/PT1000_sensor.kicad_sch (KiCad schematic)
At the start: 18 parts, among them Q1 BC546, U1 LTC2055

Commit message: created a pcb and sends it of
Parts:
- added C10, C9: 100nF, Capacitor_SMD:C_0805_2012Metric, symbol Device:C
- added J1, J2, J3: Conn_01x02_Pin, Connector_PinHeader_1.00mm:PinHeader_1x02_P1.00mm_Vertical, symbol Connector:Conn_01x02_Pin
- added R4: 160K, Resistor_SMD:R_0805_2012Metric, symbol Device:R
- added R6: 62, Resistor_SMD:R_0805_2012Metric, symbol Device:R
- added R7: 510, Resistor_SMD:R_0805_2012Metric, symbol Device:R
- R1: value 972 -> 910
- R3: value 16.5k -> 16k
Connections:
- net +3.3V: now also J2.1 (Pin_1); no longer C6.1
- net +5V: now also C6.1, C9.1, J1.1 (Pin_1)
- net GND: now also C10.2, C9.2, J1.2 (Pin_2), J2.2 (Pin_2), J3.1 (Pin_1)
- net at AD2.2 (Rg): now also R3.2; no longer R3.1
- net at AD2.3 (Rg): now also R7.2; no longer R3.2
- net at AD2.7: now also R4.1
- net at U1.5 (+): now also C10.1, R4.2
- net at U1.6 (-): now also U1.7, J3.2 (Pin_2)
- net at AD1.2 (Rg): now also R1.2; no longer R1.1
- net at AD1.3 (Rg): now also R6.2; no longer R1.2
- new net: R3.1, R7.1
- new net: R1.1, R6.1
Other:
- moved on the sheet: AD2, C6, R1, R3, U1B
